Commit message: done till simulation lidar

File: isro_rover_/description/robot_core.xacro (robot description, xacro)
@@ -15,4 +15,11 @@
     </material>
     <link name="base_link">
+    </link>
+    <joint name="base_footprint_joint" type="fixed">
+        <parent link="base_link"/>
+        <child link="base_footprint"/>
+        <origin xyz="0 0 0" rpy="0 0 0"/>
+    </joint>
+    <link name="base_footprint">
     </link>
     <joint name="chassis_joint" type="fixed">
